File: Ontwerpopdracht 1/PCB/Horloge/Horloge.kicad_pcb (KiCad board)
At the start: 2 copper layers, 12 parts

Commit message: schema
Parts:
- removed the REF** at (86.0, 73.7)
- removed the REF** at (116.8, 127.0)
- removed the REF** at (86.0, 109.2)
- removed the REF** at (81.3, 91.4)
- removed the REF** at (99.1, 122.3)
- removed the REF** at (152.4, 91.4)
- removed the REF** at (147.6, 109.2)
- removed the REF** at (147.6, 73.6)
- removed the REF** at (134.6, 60.6)
- removed the REF** at (116.8, 55.9)
- removed the REF** at (134.6, 122.2)
- removed the REF** at (99.0, 60.7)
- added REF**: SW_EVQ-P7L01P, EVQ-P7L01P:SW_EVQ-P7L01P, F.Cu at (154.9, 91.4)
- added REF**: SW_EVQ-P7L01P, EVQ-P7L01P:SW_EVQ-P7L01P, F.Cu at (154.4, 98.1)
- added REF**: LED_WS2812B-2020_PLCC4_2.0x2.0mm, LED_SMD:LED_WS2812B-2020_PLCC4_2.0x2.0mm, F.Cu at (116.8, 53.3)
- added REF**: SW_EVQ-P7L01P, EVQ-P7L01P:SW_EVQ-P7L01P, F.Cu at (154.4, 84.8)
