File: Ontwerpopdracht 1/PCB/Horloge/Horloge.kicad_pcb (KiCad board)
At the start: 2 copper layers, 41 parts, among them J1 Conn_01x03, J2 Conn_01x01, J3 Conn_01x01, Q1 BSS138, U1 TPS613222ADBVT, U2 ATTINY414-SSF, Y1 FX135A-327

Commit message: pcb
Parts:
- removed J2, J3: Conn_01x01, Connector_PinHeader_2.00mm:PinHeader_1x01_P2.00mm_Vertical
- added BT1: S8421-45R, S8421-45R:BAT_S8421-45R, B.Cu at (83.7, 98.8)
- added R4: 1k, Resistor_SMD:R_0805_2012Metric_Pad1.20x1.40mm_HandSolder, F.Cu at (84.1, 95.9)
- added TP1: Data uren, TestPoint:TestPoint_Pad_1.5x1.5mm, F.Cu at (77.5, 85.7)
- added TP2: Data min, TestPoint:TestPoint_Pad_1.5x1.5mm, F.Cu at (90.2, 87.0)
- added TP3: 5V TP, TestPoint:TestPoint_Pad_1.5x1.5mm, B.Cu at (78.1, 81.3)
- added TP4: BT1, TestPoint:TestPoint_Pad_1.5x1.5mm, B.Cu at (96.5, 104.1)
- added TP5: BT2, TestPoint:TestPoint_Pad_1.5x1.5mm, B.Cu at (99.1, 95.2)
- added TP6: BT3, TestPoint:TestPoint_Pad_1.5x1.5mm, B.Cu at (98.4, 87.6)
- R1, R2, R3, S1, S2, S3: moved to B.Cu
- moved D9 65.3 mm to (68.7, 100.2), turned to -60 degrees
- moved R1 63.8 mm to (94.6, 101.0)
- moved R2 59.5 mm to (96.5, 92.7)
- moved S2 58.5 mm to (102.2, 91.4), turned to -90 degrees
- moved D7 58.0 mm to (83.8, 108.9)
- moved D8 57.0 mm to (75.1, 106.6), turned to -30 degrees
- moved S1 56.7 mm to (99.8, 100.6), turned to -120 degrees
- moved R3 53.1 mm to (95.9, 84.5)
- moved D10 50.6 mm to (66.3, 91.4), turned to -90 degrees
- moved D24 46.4 mm to (77.1, 79.7), turned to -150 degrees
- moved D11 45.9 mm to (68.7, 82.7), turned to -120 degrees
- moved D14 44.4 mm to (90.6, 79.7), turned to 150 degrees
- moved S3 44.1 mm to (99.8, 82.2), turned to -60 degrees
- moved D12 41.9 mm to (75.1, 76.3), turned to -150 degrees
- moved D23 40.8 mm to (72.1, 84.7), turned to -120 degrees
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Connections:
- net VSS renamed VDD
- U2 pad 11: LEDS MINUTEN -> unconnected-(U2-Pad11)
- U2 pad 12: LEDS UREN -> unconnected-(U2-Pad12)
- U2 pad 13: unconnected-(U2-Pad13) -> LEDS MINUTEN
- U2 pad 3: unconnected-(U2-Pad3) -> LEDS UREN
Routing:
- net VCC: track 0.00 -> 13.2 mm
- net KNOP LINKS: track 0.00 -> 9.79 mm
- net KNOP MIDDEN: track 0.00 -> 8.81 mm
- net KNOP RECHTS: track 0.00 -> 7.18 mm
- net +5V: track 0.00 -> 6.27 mm
- net Net-(L1-Pad2): track 0.00 -> 2.29 mm
- added copper zone on B.Cu, net GND
- added copper zone on F.Cu, net GND
Other:
- board outline added: 40 x 40 mm

Commit message: pcb klaar
Parts:
- moved TP4 6.35 mm to (96.5, 97.8)
- moved TP3 6.25 mm to (83.8, 78.7)
- moved C1 4.44 mm to (77.5, 78.7)
- moved U1 4.44 mm to (77.5, 81.9)
- moved TP5 2.84 mm to (96.5, 94.0)
- moved TP1 2.62 mm to (78.1, 88.3)
- moved R2 2.51 mm to (94.9, 90.8)
- moved J1 2.10 mm to (82.8, 82.5), turned to 90 degrees
- moved R1 1.27 mm to (95.9, 101.0), turned to 90 degrees
- moved TP2 0.64 mm to (89.5, 87.0)
Routing:
- net VDD: track 0.00 -> 192.6 mm
- net +5V: track 6.27 -> 73.1 mm, vias 0 -> 4
- net KNOP RECHTS: track 7.18 -> 39.3 mm, vias 0 -> 1
- net KNOP MIDDEN: track 8.81 -> 38.6 mm, vias 0 -> 1
- net LEDS UREN: track 0.00 -> 19.3 mm
- net KNOP LINKS: track 9.79 -> 29.0 mm, vias 0 -> 1
- net LEDS MINUTEN: track 0.00 -> 14.9 mm
- net UDPI: track 0.00 -> 9.56 mm
- net Net-(D1-Pad2): track 0.00 -> 7.99 mm
- net Net-(D7-Pad2): track 0.00 -> 7.99 mm
- net Net-(D10-Pad2): track 0.00 -> 7.99 mm
- net Net-(D4-Pad2): track 0.00 -> 7.97 mm
- net LEDS UIT: track 0.00 -> 7.80 mm
- net Net-(D11-Pad2): track 0.00 -> 7.74 mm
- net Net-(D5-Pad2): track 0.00 -> 7.73 mm
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
Commit message: pcb
Parts:
- added TP7: 3V, TestPoint:TestPoint_Pad_1.5x1.5mm, B.Cu at (88.9, 82.5)
- added TP8: LEDSW, TestPoint:TestPoint_Pad_1.5x1.5mm, F.Cu at (80.6, 99.1)
- TP3: value 5V TP -> 5V
Routing:
- net VCC: track 13.2 -> 19.8 mm
- net VDD: track 192.6 -> 196.4 mm
- net KNOP MIDDEN: track 38.6 -> 37.1 mm
- net +5V: track 73.1 -> 71.6 mm
- net KNOP LINKS: track 29.0 -> 28.1 mm
- net KNOP RECHTS: track 39.3 -> 38.6 mm

Commit message: pcb finaal + code
Parts:
- J1: footprint Connector_PinHeader_1.00mm:PinHeader_1x03_P1.00mm_Vertical -> Connector_PinHeader_2.54mm:PinHeader_1x03_P2.54mm_Vertical
- moved J1 1.54 mm to (81.3, 82.5)
Routing:
- net +5V: track 71.6 -> 69.1 mm
- net VCC: track 19.8 -> 20.9 mm
- net LEDS MINUTEN: track 14.9 -> 15.6 mm
