File: Ontwerpopdracht 1/PCB/Horloge/Horloge.kicad_sch (KiCad schematic)
At the start: 47 parts, among them J1 Conn_01x03, Q1 BSS138, U1 TPS613222ADBVT, U2 ATTINY414-SSF, Y1 FX135A-327

Commit message: pcb
Parts:
- removed BT1: Battery_Cell, symbol Device:Battery_Cell
- added BT1: S8421-45R, S8421-45R:BAT_S8421-45R, symbol S8421-45R:S8421-45R
- R4: value 4k7 -> 1k
- TP1, TP2, TP4, TP5, TP6: footprint (none) -> TestPoint:TestPoint_Pad_1.5x1.5mm
- TP3: value 5V -> 5V TP; footprint (none) -> TestPoint:TestPoint_Pad_1.5x1.5mm
Connections:
- net GND: now also BT1.-
- net VCC: now also BT1.+
Changed lines of the file:
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@@
-    (stroke (width 0) (type default) (color 0 0 0 0))
-  )
-  (wire (pts (xy 19.05 35.56) (xy 19.05 39.37))
     (stroke (width 0) (type default) (color 0 0 0 0))
   )
@@
   )
   (wire (pts (xy 218.44 39.37) (xy 219.71 39.37))
-    (stroke (width 0) (type default) (color 0 0 0 0))
-  )
-  (wire (pts (xy 19.05 24.13) (xy 19.05 27.94))
     (stroke (width 0) (type default) (color 0 0 0 0))
   )
@@
       (effects (font (size 1.27 1.27)) (justify left))
     )
-    (property "Value" "5V" (id 1) (at 96.52 27.94 90)
-      (effects (font (size 1.27 1.27)) (justify left))
-    )
-    (property "Footprint" "" (id 2) (at 91.44 31.75 0)
+    (property "Value" "5V TP" (id 1) (at 95.25 27.94 90)
+      (effects (font (size 1.27 1.27)) (justify left))
+    )
+    (property "Footprint" "TestPoint:TestPoint_Pad_1.5x1.5mm" (id 2) (at 91.44 31.75 0)
       (effects (font (size 1.27 1.27)) hide)
     )
@@
     (pin "4")
   )
-  (symbol (lib_id "Device:Battery_Cell") (at 19.05 33.02 0) (unit 1)
-    (in_bom yes) (on_board yes) (fields_autoplaced)
-    (property "Reference" "BT1" (id 0) (at 22.86 29.7179 0)
-      (effects (font (size 1.27 1.27)) (justify left))
-    )
-    (property "Value" "Battery_Cell" (id 1) (at 22.86 32.2579 0)
-      (effects (font (size 1.27 1.27)) (justify left))
-    )
-    (property "Footprint" "" (id 2) (at 19.05 31.496 90)
-      (effects (font (size 1.27 1.27)) hide)
-    )
-    (property "Datasheet" "~" (id 3) (at 19.05 31.496 90)
-      (effects (font (size 1.27 1.27)) hide)
-    )
-    (pin "1")
-    (pin "2")
-  )
   (symbol (lib_id "LED:WS2812B") (at 135.89 114.3 0) (unit 1)
     (in_bom yes) (on_board yes)
@@
       (effects (font (size 1.27 1.27)) (justify left))
     )
-    (property "Footprint" "" (id 2) (at 223.52 39.37 0)
+    (property "Footprint" "TestPoint:TestPoint_Pad_1.5x1.5mm" (id 2) (at 223.52 39.37 0)
       (effects (font (size 1.27 1.27)) hide)
     )
@@
       (effects (font (size 1.27 1.27)) (justify left))
     )
-    (property "Footprint" "" (id 2) (at 223.52 82.55 0)
+    (property "Footprint" "TestPoint:TestPoint_Pad_1.5x1.5mm" (id 2) (at 223.52 82.55 0)
       (effects (font (size 1.27 1.27)) hide)
     )
@@
   (symbol (lib_id "power:VDD") (at 269.24 24.13 0) (mirror y) (unit 1)
     (in_bom yes) (on_board yes)
-    (property "Reference" "#PWR?" (id 0) (at 269.24 27.94 0)
+    (property "Reference" "#PWR0101" (id 0) (at 269.24 27.94 0)
       (effects (font (size 1.27 1.27)) hide)
     )
@@
       (effects (font (size 1.27 1.27)) (justify left))
     )
-    (property "Footprint" "" (id 2) (at 17.78 109.22 0)
+    (property "Footprint" "TestPoint:TestPoint_Pad_1.5x1.5mm" (id 2) (at 17.78 109.22 0)
       (effects (font (size 1.27 1.27)) hide)
     )
@@
       (effects (font (size 1.27 1.27)) (justify left))
     )
-    (property "Footprint" "" (id 2) (at 17.78 144.78 0)
+    (property "Footprint" "TestPoint:TestPoint_Pad_1.5x1.5mm" (id 2) (at 17.78 144.78 0)
       (effects (font (size 1.27 1.27)) hide)
     )
@@
       (effects (font (size 1.27 1.27)) (justify left))
     )
-    (property "Footprint" "" (id 2) (at 223.52 60.96 0)
+    (property "Footprint" "TestPoint:TestPoint_Pad_1.5x1.5mm" (id 2) (at 223.52 60.96 0)
       (effects (font (size 1.27 1.27)) hide)
     )
@@
     (pin "4")
   )
+  (symbol (lib_id "S8421-45R:S8421-45R") (at 19.05 31.75 270) (unit 1)
+    (in_bom yes) (on_board yes) (fields_autoplaced)
+    (property "Reference" "BT1" (id 0) (at 22.86 29.8449 90)
+      (effects (font (size 1.27 1.27)) (justify left))
+    )
+    (property "Value" "S8421-45R" (id 1) (at 22.86 32.3849 90)
+      (effects (font (size 1.27 1.27)) (justify left))
+    )
+    (property "Footprint" "S8421-45R:BAT_S8421-45R" (id 2) (at 19.05 31.75 0)
+      (effects (font (size 1.27 1.27)) (justify bottom) hide)
+    )
+    (property "Datasheet" "" (id 3) (at 19.05 31.75 0)
+      (effects (font (size 1.27 1.27)) hide)
+    )
+    (property "MAXIMUM_PACKAGE_HIEGHT" "5.3mm" (id 4) (at 19.05 31.75 0)
+      (effects (font (size 1.27 1.27)) (justify bottom) hide)
+    )
+    (property "MANUFACTURER" "Harwin" (id 5) (at 19.05 31.75 0)
+      (effects (font (size 1.27 1.27)) (justify bottom) hide)
+    )
+    (property "PARTREV" "5" (id 6) (at 19.05 31.75 0)
+      (effects (font (size 1.27 1.27)) (justify bottom) hide)
+    )
+    (property "STANDARD" "Manufacturer Recommendations" (id 7) (at 19.05 31.75 0)
+      (effects (font (size 1.27 1.27)) (justify bottom) hide)
+    )
+    (pin "+")
+    (pin "-")
+  )
   (symbol (lib_id "power:GND") (at 19.05 39.37 0) (unit 1)
     (in_bom yes) (on_board yes)
@@
     (in_bom yes) (on_board yes)
     (property "Reference" "R4" (id 0) (at 252.73 31.75 90))
-    (property "Value" "4k7" (id 1) (at 257.81 31.75 90)
-      (effects (font (size 1.27 1.27)) hide)
-    )
+    (property "Value" "1k" (id 1) (at 257.81 31.75 90))
     (property "Footprint" "Resistor_SMD:R_0805_2012Metric_Pad1.20x1.40mm_HandSolder" (id 2) (at 257.048 31.75 90)
       (effects (font (size 1.27 1.27)) hide)
@@
   (symbol (lib_id "power:VDD") (at 27.94 104.14 0) (unit 1)
     (in_bom yes) (on_board yes)
-    (property "Reference" "#PWR?" (id 0) (at 27.94 107.95 0)
+    (property "Reference" "#PWR0102" (id 0) (at 27.94 107.95 0)
       (effects (font (size 1.27 1.27)) hide)
     )
@@
   (symbol (lib_id "power:VDD") (at 27.94 139.7 0) (unit 1)
     (in_bom yes) (on_board yes)
-    (property "Reference" "#PWR?" (id 0) (at 27.94 143.51 0)
+    (property "Reference" "#PWR0103" (id 0) (at 27.94 143.51 0)
       (effects (font (size 1.27 1.27)) hide)
     )
@@
       (reference "#PWR035") (unit 1) (value "+5V") (footprint "")
     )
+    (path "/6cbbf477-cbfc-493f-ac49-a07c9d283098"
+      (reference "#PWR0101") (unit 1) (value "VDD") (footprint "")
+    )
+    (path "/e022f9a2-9ca5-447d-a3c0-cf8556f85686"
+      (reference "#PWR0102") (unit 1) (value "VDD") (footprint "")
+    )
+    (path "/fb658080-d24a-4a9e-8e24-b28894de43fd"
+      (reference "#PWR0103") (unit 1) (value "VDD") (footprint "")
+    )
     (path "/91a422fb-7118-4a8c-80f3-79b1db52358e"
       (reference "#PWR0115") (unit 1) (value "GND") (footprint "")
@@
       (reference "#PWR0119") (unit 1) (value "GND") (footprint "")
     )
-    (path "/6cbbf477-cbfc-493f-ac49-a07c9d283098"
-      (reference "#PWR?") (unit 1) (value "VDD") (footprint "")
-    )
-    (path "/e022f9a2-9ca5-447d-a3c0-cf8556f85686"
-      (reference "#PWR?") (unit 1) (value "VDD") (footprint "")
-    )
-    (path "/fb658080-d24a-4a9e-8e24-b28894de43fd"
-      (reference "#PWR?") (unit 1) (value "VDD") (footprint "")
-    )
-    (path "/1b070be4-7e29-4e18-85f3-746e2b378b88"
-      (reference "BT1") (unit 1) (value "Battery_Cell") (footprint "")
+    (path "/b3b2d609-99d2-45ed-b735-7b0561a03e72"
+      (reference "BT1") (unit 1) (value "S8421-45R") (footprint "S8421-45R:BAT_S8421-45R")
     )
     (path "/d7e56d45-a657-43fb-bc8b-670c5cd57934"
@@
     )
     (path "/deb6f103-7bc7-4e9c-8481-3fae47a726dc"
-      (reference "R4") (unit 1) (value "4k7") (footprint "Resistor_SMD:R_0805_2012Metric_Pad1.20x1.40mm_HandSolder")
+      (reference "R4") (unit 1) (value "1k") (footprint "Resistor_SMD:R_0805_2012Metric_Pad1.20x1.40mm_HandSolder")
     )
     (path "/42ec860a-394c-4659-94f0-852b817b320c"
@@
     )
     (path "/798c1536-a120-4a30-b1b2-9a14c65e8257"
-      (reference "TP1") (unit 1) (value "Data uren") (footprint "")
+      (reference "TP1") (unit 1) (value "Data uren") (footprint "TestPoint:TestPoint_Pad_1.5x1.5mm")
     )
     (path "/9223ef91-e53b-43f2-bb61-2ddb9a31485c"
-      (reference "TP2") (unit 1) (value "Data min") (footprint "")
+      (reference "TP2") (unit 1) (value "Data min") (footprint "TestPoint:TestPoint_Pad_1.5x1.5mm")
     )
     (path "/08dd50c7-52ba-4b85-ac1e-70c26403dd00"
-      (reference "TP3") (unit 1) (value "5V") (footprint "")
+      (reference "TP3") (unit 1) (value "5V TP") (footprint "TestPoint:TestPoint_Pad_1.5x1.5mm")
     )
     (path "/37271720-d97c-4e51-ac0f-3ee808ef91a7"
-      (reference "TP4") (unit 1) (value "BT1") (footprint "")
+      (reference "TP4") (unit 1) (value "BT1") (footprint "TestPoint:TestPoint_Pad_1.5x1.5mm")
     )
     (path "/980010d4-48e5-4897-b229-42d0c9746642"
-      (reference "TP5") (unit 1) (value "BT2") (footprint "")
+      (reference "TP5") (unit 1) (value "BT2") (footprint "TestPoint:TestPoint_Pad_1.5x1.5mm")
     )
     (path "/5fafa8d5-747a-47f3-aa91-8261073502a9"
-      (reference "TP6") (unit 1) (value "BT3") (footprint "")
+      (reference "TP6") (unit 1) (value "BT3") (footprint "TestPoint:TestPoint_Pad_1.5x1.5mm")
     )
     (path "/66083f19-7996-4877-9c17-f60ae0bcb5db"

Commit message: pcb
Parts:
- added TP7: 3V, TestPoint:TestPoint_Pad_1.5x1.5mm, symbol Connector:TestPoint
- added TP8: LEDSW, TestPoint:TestPoint_Pad_1.5x1.5mm, symbol Connector:TestPoint
- TP3: value 5V TP -> 5V
Connections:
- net VCC: now also TP7.1
- net VDD: now also TP8.1
Changed lines of the file:
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@@
   (junction (at 49.53 105.41) (diameter 0) (color 0 0 0 0)
   )
+  (junction (at 269.24 26.67) (diameter 0) (color 0 0 0 0)
+  )
   (junction (at 76.2 58.42) (diameter 0) (color 0 0 0 0)
   )
@@
   (junction (at 114.3 105.41) (diameter 0) (color 0 0 0 0)
   )
+  (junction (at 40.64 26.67) (diameter 0) (color 0 0 0 0)
+  )
   (junction (at 27.94 140.97) (diameter 0) (color 0 0 0 0)
   )
@@
     (stroke (width 0) (type default) (color 0 0 0 0))
   )
-  (wire (pts (xy 40.64 31.75) (xy 40.64 24.13))
+  (wire (pts (xy 40.64 31.75) (xy 40.64 26.67))
     (stroke (width 0) (type default) (color 0 0 0 0))
   )
@@
   )
   (wire (pts (xy 27.94 142.24) (xy 27.94 140.97))
+    (stroke (width 0) (type default) (color 0 0 0 0))
+  )
+  (wire (pts (xy 40.64 26.67) (xy 40.64 24.13))
     (stroke (width 0) (type default) (color 0 0 0 0))
   )
@@
       (effects (font (size 1.27 1.27)) (justify left))
     )
-    (property "Value" "5V TP" (id 1) (at 95.25 27.94 90)
+    (property "Value" "5V" (id 1) (at 96.52 27.94 90)
       (effects (font (size 1.27 1.27)) (justify left))
     )
@@
     (pin "2")
     (pin "4")
+  )
+  (symbol (lib_id "Connector:TestPoint") (at 269.24 26.67 180) (unit 1)
+    (in_bom yes) (on_board yes)
+    (property "Reference" "TP8" (id 0) (at 267.97 31.75 0)
+      (effects (font (size 1.27 1.27)) (justify left))
+    )
+    (property "Value" "LEDSW" (id 1) (at 270.51 34.29 0)
+      (effects (font (size 1.27 1.27)) (justify left))
+    )
+    (property "Footprint" "TestPoint:TestPoint_Pad_1.5x1.5mm" (id 2) (at 264.16 26.67 0)
+      (effects (font (size 1.27 1.27)) hide)
+    )
+    (property "Datasheet" "~" (id 3) (at 264.16 26.67 0)
+      (effects (font (size 1.27 1.27)) hide)
+    )
+    (pin "1")
   )
   (symbol (lib_id "power:VDD") (at 269.24 24.13 0) (mirror y) (unit 1)
@@
     (pin "4")
   )
+  (symbol (lib_id "Connector:TestPoint") (at 40.64 26.67 90) (unit 1)
+    (in_bom yes) (on_board yes)
+    (property "Reference" "TP7" (id 0) (at 34.29 27.94 90)
+      (effects (font (size 1.27 1.27)) (justify left))
+    )
+    (property "Value" "3V" (id 1) (at 34.29 25.4 90)
+      (effects (font (size 1.27 1.27)) (justify left))
+    )
+    (property "Footprint" "TestPoint:TestPoint_Pad_1.5x1.5mm" (id 2) (at 40.64 21.59 0)
+      (effects (font (size 1.27 1.27)) hide)
+    )
+    (property "Datasheet" "~" (id 3) (at 40.64 21.59 0)
+      (effects (font (size 1.27 1.27)) hide)
+    )
+    (pin "1")
+  )
   (symbol (lib_id "LED:WS2812B") (at 157.48 149.86 0) (unit 1)
     (in_bom yes) (on_board yes) (fields_autoplaced)
@@
     )
     (path "/08dd50c7-52ba-4b85-ac1e-70c26403dd00"
-      (reference "TP3") (unit 1) (value "5V TP") (footprint "TestPoint:TestPoint_Pad_1.5x1.5mm")
+      (reference "TP3") (unit 1) (value "5V") (footprint "TestPoint:TestPoint_Pad_1.5x1.5mm")
     )
     (path "/37271720-d97c-4e51-ac0f-3ee808ef91a7"
@@
       (reference "TP6") (unit 1) (value "BT3") (footprint "TestPoint:TestPoint_Pad_1.5x1.5mm")
     )
+    (path "/d04667bb-5f84-4d14-8b13-225803bcc4f8"
+      (reference "TP7") (unit 1) (value "3V") (footprint "TestPoint:TestPoint_Pad_1.5x1.5mm")
+    )
+    (path "/67429933-4b12-40cb-84d5-80079e0513ea"
+      (reference "TP8") (unit 1) (value "LEDSW") (footprint "TestPoint:TestPoint_Pad_1.5x1.5mm")
+    )
     (path "/66083f19-7996-4877-9c17-f60ae0bcb5db"

Commit message: pcb finaal + code
Parts:
- J1: footprint Connector_PinHeader_1.00mm:PinHeader_1x03_P1.00mm_Vertical -> Connector_PinHeader_2.54mm:PinHeader_1x03_P2.54mm_Vertical
Changed lines of the file:
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@@
       (effects (font (size 1.27 1.27)) (justify left) hide)
     )
-    (property "Footprint" "Connector_PinHeader_1.00mm:PinHeader_1x03_P1.00mm_Vertical" (id 2) (at 31.75 57.15 0)
+    (property "Footprint" "Connector_PinHeader_2.54mm:PinHeader_1x03_P2.54mm_Vertical" (id 2) (at 31.75 57.15 0)
       (effects (font (size 1.27 1.27)) hide)
     )
@@
     )
     (path "/35d1ac95-96f8-4902-9ae0-f86acb453796"
-      (reference "J1") (unit 1) (value "Conn_01x03") (footprint "Connector_PinHeader_1.00mm:PinHeader_1x03_P1.00mm_Vertical")
+      (reference "J1") (unit 1) (value "Conn_01x03") (footprint "Connector_PinHeader_2.54mm:PinHeader_1x03_P2.54mm_Vertical")
     )
     (path "/e8b02372-df70-4a53-bb2e-192ce2085ac9"

Commit message: pcb macropad klaar
Connections:
- net GND: now also D1.2 (VSS), D10.2 (VSS), D11.2 (VSS), D12.2 (VSS), D13.2 (VSS), D14.2 (VSS), D15.2 (VSS), D16.2 (VSS), D17.2 (VSS), D18.2 (VSS), D19.2 (VSS), D2.2 (VSS), D20.2 (VSS), D21.2 (VSS), D22.2 (VSS), D23.2 (VSS), D24.2 (VSS), D3.2 (VSS), D4.2 (VSS), D5.2 (VSS), D6.2 (VSS), D7.2 (VSS), D8.2 (VSS), D9.2 (VSS); no longer D1.3 (VSS), D10.3 (VSS), D11.3 (VSS), D12.3 (VSS), D13.3 (VSS), D14.3 (VSS), D15.3 (VSS), D16.3 (VSS), D17.3 (VSS), D18.3 (VSS), D19.3 (VSS), D2.3 (VSS), D20.3 (VSS), D21.3 (VSS), D22.3 (VSS), D23.3 (VSS), D24.3 (VSS), D3.3 (VSS), D4.3 (VSS), D5.3 (VSS), D6.3 (VSS), D7.3 (VSS), D8.3 (VSS), D9.3 (VSS)
- net LEDS MINUTEN: now also D13.3 (DIN); no longer D13.4 (DIN)
- net LEDS UREN: now also D1.3 (DIN); no longer D1.4 (DIN)
- net VDD: now also D1.4 (VDD), D10.4 (VDD), D11.4 (VDD), D12.4 (VDD), D13.4 (VDD), D14.4 (VDD), D15.4 (VDD), D16.4 (VDD), D17.4 (VDD), D18.4 (VDD), D19.4 (VDD), D2.4 (VDD), D20.4 (VDD), D21.4 (VDD), D22.4 (VDD), D23.4 (VDD), D24.4 (VDD), D3.4 (VDD), D4.4 (VDD), D5.4 (VDD), D6.4 (VDD), D7.4 (VDD), D8.4 (VDD), D9.4 (VDD); no longer D1.1 (VDD), D10.1 (VDD), D11.1 (VDD), D12.1 (VDD), D13.1 (VDD), D14.1 (VDD), D15.1 (VDD), D16.1 (VDD), D17.1 (VDD), D18.1 (VDD), D19.1 (VDD), D2.1 (VDD), D20.1 (VDD), D21.1 (VDD), D22.1 (VDD), D23.1 (VDD), D24.1 (VDD), D3.1 (VDD), D4.1 (VDD), D5.1 (VDD), D6.1 (VDD), D7.1 (VDD), D8.1 (VDD), D9.1 (VDD)
- new net: D20.1 (DOUT), D21.3 (DIN)
- new net: D19.1 (DOUT), D20.3 (DIN)
- new net: D4.1 (DOUT), D5.3 (DIN)
- new net: D3.1 (DOUT), D4.3 (DIN)
- new net: D11.1 (DOUT), D12.3 (DIN)
- new net: D10.1 (DOUT), D11.3 (DIN)
- new net: D23.1 (DOUT), D24.3 (DIN)
- new net: D18.1 (DOUT), D19.3 (DIN)
- new net: D17.1 (DOUT), D18.3 (DIN)
- new net: D2.1 (DOUT), D3.3 (DIN)
- new net: D1.1 (DOUT), D2.3 (DIN)
- new net: D22.1 (DOUT), D23.3 (DIN)
- new net: D21.1 (DOUT), D22.3 (DIN)
- new net: D7.1 (DOUT), D8.3 (DIN)
- new net: D6.1 (DOUT), D7.3 (DIN)
- new net: D13.1 (DOUT), D14.3 (DIN)
- new net: D16.1 (DOUT), D17.3 (DIN)
- new net: D14.1 (DOUT), D15.3 (DIN)
- new net: D10.3 (DIN), D9.1 (DOUT)
- new net: D8.1 (DOUT), D9.3 (DIN)
- new net: D5.1 (DOUT), D6.3 (DIN)
- new net: D15.1 (DOUT), D16.3 (DIN)
