File: Ontwerpopdracht 2/PCB/Macropad/Macropad.kicad_pcb (KiCad board)
At the start: 2 copper layers, 59.7 x 59.7 mm, 15 parts, among them IC1 PEC12R-4220F-S0024, IC2 PEC12R-4220F-S0024

Commit message: pcb
Parts:
- added C1: 0.01uF, Capacitor_SMD:C_0805_2012Metric_Pad1.18x1.45mm_HandSolder, F.Cu at (113.0, 29.4)
- added C2: 0.01uF, Capacitor_SMD:C_0805_2012Metric_Pad1.18x1.45mm_HandSolder, F.Cu at (113.0, 32.4)
- added C3: 0.01uF, Capacitor_SMD:C_0805_2012Metric_Pad1.18x1.45mm_HandSolder, F.Cu at (113.0, 35.4)
- added C4: 0.01uF, Capacitor_SMD:C_0805_2012Metric_Pad1.18x1.45mm_HandSolder, F.Cu at (113.0, 38.4)
- added H1: MountingHole_Pad, MountingHole:MountingHole_2.2mm_M2_Pad_Via, F.Cu at (61.0, 88.8)
- added H2: MountingHole_Pad, MountingHole:MountingHole_2.2mm_M2_Pad_Via, F.Cu at (81.0, 88.8)
- added H3: MountingHole_Pad, MountingHole:MountingHole_2.2mm_M2_Pad_Via, F.Cu at (85.8, 53.0)
- added H4: MountingHole_Pad, MountingHole:MountingHole_2.2mm_M2_Pad_Via, F.Cu at (56.2, 53.0)
- added R1: 10K, Resistor_SMD:R_0805_2012Metric_Pad1.20x1.40mm_HandSolder, F.Cu at (108.2, 29.4)
- added R2: 10K, Resistor_SMD:R_0805_2012Metric_Pad1.20x1.40mm_HandSolder, F.Cu at (108.2, 32.3)
- added R3: 10K, Resistor_SMD:R_0805_2012Metric_Pad1.20x1.40mm_HandSolder, F.Cu at (108.2, 35.2)
- added R4: 10K, Resistor_SMD:R_0805_2012Metric_Pad1.20x1.40mm_HandSolder, F.Cu at (108.2, 38.2)
- added R5: 10K, Resistor_SMD:R_0805_2012Metric_Pad1.20x1.40mm_HandSolder, F.Cu at (84.2, 46.6)
- added R6: 10K, Resistor_SMD:R_0805_2012Metric_Pad1.20x1.40mm_HandSolder, F.Cu at (85.0, 34.2)
- added R7: 10K, Resistor_SMD:R_0805_2012Metric_Pad1.20x1.40mm_HandSolder, F.Cu at (98.8, 52.4)
- added R8: 10K, Resistor_SMD:R_0805_2012Metric_Pad1.20x1.40mm_HandSolder, F.Cu at (94.8, 52.4)
- moved D2 59.1 mm to (52.4, 75.4)
- moved D1 57.4 mm to (52.5, 55.0)
- moved D3 38.2 mm to (72.8, 55.0)
- moved D4 38.1 mm to (72.8, 75.4)
- moved S5 29.1 mm to (93.9, 57.9)
- moved S2 28.6 mm to (53.1, 78.3)
- moved D5 21.8 mm to (93.2, 55.0)
- moved S4 20.8 mm to (73.5, 78.3)
- moved S3 19.8 mm to (73.5, 57.9)
- moved D6 17.1 mm to (93.2, 75.4)
- moved IC2 0.78 mm to (89.5, 34.9)
- moved IC1 0.72 mm to (47.5, 34.9)
- moved S6 0.63 mm to (93.9, 78.3)
- moved S1 0.46 mm to (53.1, 57.9)
- moved A1 0.41 mm to (70.9, 58.4)
Connections:
- A1 pad 1: unconnected-(A1-GP0-Pad1) -> RIJ1
- A1 pad 2: unconnected-(A1-GP1-Pad2) -> RIJ2
- A1 pad 36: unconnected-(A1-3V3_OUT-Pad36) -> +3V3
- A1 pad 4: unconnected-(A1-GP2-Pad4) -> KOLOM1
- A1 pad 5: unconnected-(A1-GP3-Pad5) -> KOLOM2
- A1 pad 6: unconnected-(A1-GP4-Pad6) -> KOLOM3
- D1 pad 1: unconnected-(D1-K-Pad1) -> KOLOM1
- D1 pad 2: unconnected-(D1-A-Pad2) -> Net-(D1-A)
- D2 pad 1: unconnected-(D2-K-Pad1) -> KOLOM1
- D2 pad 2: unconnected-(D2-A-Pad2) -> Net-(D2-A)
- D3 pad 1: unconnected-(D3-K-Pad1) -> KOLOM2
- D3 pad 2: unconnected-(D3-A-Pad2) -> Net-(D3-A)
- D4 pad 1: unconnected-(D4-K-Pad1) -> KOLOM2
- D4 pad 2: unconnected-(D4-A-Pad2) -> Net-(D4-A)
- D5 pad 1: unconnected-(D5-K-Pad1) -> KOLOM3
- D5 pad 2: unconnected-(D5-A-Pad2) -> Net-(D5-A)
- D6 pad 1: unconnected-(D6-K-Pad1) -> KOLOM3
- D6 pad 2: unconnected-(D6-A-Pad2) -> Net-(D6-A)
- IC1 pad 1: unconnected-(IC1-Pad1) -> Net-(IC1-Pad1)
- IC1 pad 2: unconnected-(IC1-Pad2) -> Net-(IC1-Pad2)
- IC1 pad A1: unconnected-(IC1-PadA1) -> ROT1A
- IC1 pad B1: unconnected-(IC1-PadB1) -> ROT1B
- IC1 pad C1: unconnected-(IC1-PadC1) -> GND
- IC2 pad 1: unconnected-(IC2-Pad1) -> Net-(IC2-Pad1)
- IC2 pad 2: unconnected-(IC2-Pad2) -> Net-(IC2-Pad2)
- IC2 pad A1: unconnected-(IC2-PadA1) -> ROT2A
- IC2 pad B1: unconnected-(IC2-PadB1) -> ROT2B
- IC2 pad C1: unconnected-(IC2-PadC1) -> GND
- S1 pad 1: unconnected-(S1-Pad1) -> Net-(D1-A)
- S1 pad 2: unconnected-(S1-Pad2) -> RIJ1
- S2 pad 1: unconnected-(S2-Pad1) -> Net-(D2-A)
- S2 pad 2: unconnected-(S2-Pad2) -> RIJ2
- S3 pad 1: unconnected-(S3-Pad1) -> Net-(D3-A)
- S3 pad 2: unconnected-(S3-Pad2) -> RIJ1
- S4 pad 1: unconnected-(S4-Pad1) -> Net-(D4-A)
- S4 pad 2: unconnected-(S4-Pad2) -> RIJ2
- S5 pad 1: unconnected-(S5-Pad1) -> Net-(D5-A)
- S5 pad 2: unconnected-(S5-Pad2) -> RIJ1
- S6 pad 1: unconnected-(S6-Pad1) -> Net-(D6-A)
- S6 pad 2: unconnected-(S6-Pad2) -> RIJ2
Routing:
- added copper zone on B.Cu, net GND
- added copper zone on F.Cu, net GND
- removed copper zone on B.Cu, net (none)
- removed copper zone on F.Cu, net (none)
Other:
- board size 59.7 x 59.7 mm -> 60 x 60 mm

Commit message: pcb klaar
Parts:
- added R10: 10K, Resistor_SMD:R_0805_2012Metric_Pad1.20x1.40mm_HandSolder, B.Cu at (43.8, 54.0)
- added R9: 10K, Resistor_SMD:R_0805_2012Metric_Pad1.20x1.40mm_HandSolder, B.Cu at (46.4, 54.0)
- C1, C2, C3, C4, D1, D2, D3, D4, D5, D6, R1, R2, R3, R4, R5, R6, R7, R8: moved to B.Cu
- moved C1 67.7 mm to (47.6, 47.0)
- moved C2 62.6 mm to (52.1, 47.0)
- moved R2 60.9 mm to (47.6, 38.1)
- moved R1 60.6 mm to (48.9, 41.9), turned to 90 degrees
- moved R3 57.2 mm to (51.4, 41.9), turned to -90 degrees
- moved R4 55.5 mm to (52.7, 38.1)
- moved C3 26.2 mm to (89.5, 47.0)
- moved C4 20.8 mm to (94.0, 47.0)
- moved R7 14.9 mm to (94.6, 38.1), turned to 0 degrees
- moved R8 10.6 mm to (93.3, 41.9), turned to -90 degrees
- moved R5 8.10 mm to (90.8, 41.9)
- moved R6 5.98 mm to (89.5, 38.1), turned to 0 degrees
- moved D5 4.84 mm to (97.2, 57.8), turned to 180 degrees
- moved D6 4.79 mm to (97.2, 78.1), turned to 180 degrees
- moved D2 4.41 mm to (55.9, 78.1), turned to 180 degrees
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Connections:
- A1 pad 1: RIJ1 -> unconnected-(A1-GP0-Pad1)
- A1 pad 14: unconnected-(A1-GP10-Pad14) -> KOLOM3
- A1 pad 15: unconnected-(A1-GP11-Pad15) -> KOLOM2
- A1 pad 16: unconnected-(A1-GP12-Pad16) -> KOLOM1
- A1 pad 2: RIJ2 -> unconnected-(A1-GP1-Pad2)
- A1 pad 21: unconnected-(A1-GP16-Pad21) -> RIJ2
- A1 pad 22: unconnected-(A1-GP17-Pad22) -> RIJ1
- A1 pad 31: unconnected-(A1-GP26-Pad31) -> ROT1A
- A1 pad 32: unconnected-(A1-GP27-Pad32) -> ROT1B
- A1 pad 4: KOLOM1 -> ROT2A
- A1 pad 5: KOLOM2 -> ROT2B
- A1 pad 6: KOLOM3 -> unconnected-(A1-GP4-Pad6)
- C2 pad 1: ROT1B -> GND
- C2 pad 2: GND -> ROT1B
- C4 pad 1: ROT2B -> GND
- C4 pad 2: GND -> ROT2B
Routing:
- net +3V3: track 0.00 -> 95.6 mm
- net RIJ1: track 0.00 -> 91.2 mm
- net RIJ2: track 0.00 -> 72.6 mm
- net KOLOM1: track 0.00 -> 50.5 mm
- net KOLOM3: track 0.00 -> 38.9 mm
- net ROT1A: track 0.00 -> 25.5 mm
- net ROT2B: track 0.00 -> 25.3 mm
- net KOLOM2: track 0.00 -> 23.7 mm
- net ROT2A: track 0.00 -> 20.7 mm
- net ROT1B: track 0.00 -> 19.1 mm
- net Net-(IC1-Pad2): track 0.00 -> 7.45 mm
- net Net-(IC2-Pad2): track 0.00 -> 7.41 mm
- net Net-(IC2-Pad1): track 0.00 -> 7.35 mm
- net Net-(IC1-Pad1): track 0.00 -> 7.31 mm
- net GND: track 0.00 -> 4.74 mm
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
Commit message: pcb klaar
Other:
- board text added: "Sten Hulsbergen"
Changed lines of the file:
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@@
   (gr_rect (start 41 33.02) (end 101 93)
     (stroke (width 0.2) (type default)) (fill none) (layer "Edge.Cuts"))
+  (gr_text "Sten \nHulsbergen\n" (at 64.77 40.005) (layer "F.SilkS")
+    (effects (font (size 1.5 1.5) (thickness 0.3) bold) (justify left bottom))
+  )
   (segment (start 60.325 62.865) (end 60.96 63.5) (width 0.25) (layer "B.Cu") (net 1))
   (segment (start 71.77 55.88) (end 67.19 60.46) (width 0.25) (layer "B.Cu") (net 1))
