File: Ontwerpopdracht 2/PCB/Macropad/Macropad.kicad_pcb (KiCad board)
At the start: 2 copper layers, 60 x 60 mm, 33 parts, among them IC1 PEC12R-4220F-S0024, IC2 PEC12R-4220F-S0024

Commit message: programatie
Parts:
- added D7: 1N4148WT, Diode_SMD:D_SOD-123, B.Cu at (69.2, 41.9)
- added D8: 1N4148WT, Diode_SMD:D_SOD-123, B.Cu at (72.4, 41.9)
- D1, D2, D3, D4, D5, D6: footprint Diode_SMD:D_SOD-523 -> Diode_SMD:D_SOD-123
- moved C1 19.9 mm to (65.4, 55.9), turned to -90 degrees
- moved C4 17.9 mm to (76.2, 45.1), turned to 90 degrees
- moved C3 14.8 mm to (76.2, 40.6), turned to 90 degrees
- moved C2 14.1 mm to (65.4, 51.4), turned to -90 degrees
- moved D5 11.9 mm to (94.0, 69.2), turned to 0 degrees
- moved D1 11.7 mm to (53.3, 69.2)
- moved D3 11.7 mm to (73.7, 69.2)
- moved R8 10.3 mm to (85.7, 48.9), turned to 180 degrees
- moved R1 10.1 mm to (56.1, 48.9), turned to 180 degrees
- moved D6 7.10 mm to (94.0, 71.8), turned to 0 degrees
- moved D4 6.84 mm to (73.7, 71.8)
- moved D2 6.84 mm to (53.3, 71.8)
- moved R5 6.75 mm to (85.7, 46.4), turned to 0 degrees
- moved R3 6.48 mm to (56.1, 46.4), turned to 0 degrees
- moved R6 4.02 mm to (90.8, 41.9), turned to 90 degrees
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Connections:
- A1 pad 6: unconnected-(A1-GP4-Pad6) -> KOLOM4
- IC1 pad 1: Net-(IC1-Pad1) -> RIJ1
- IC1 pad 2: Net-(IC1-Pad2) -> Net-(D7-A)
- IC1 pad A1: ROT1A -> Net-(IC1-PadA1)
- IC1 pad B1: ROT1B -> Net-(IC1-PadB1)
- IC2 pad 1: Net-(IC2-Pad1) -> RIJ2
- IC2 pad 2: Net-(IC2-Pad2) -> Net-(D8-A)
- IC2 pad A1: ROT2A -> Net-(IC2-PadA1)
- IC2 pad B1: ROT2B -> Net-(IC2-PadB1)
- R1 pad 2: Net-(IC1-Pad1) -> Net-(IC1-PadA1)
- R2 pad 1: Net-(IC1-Pad1) -> Net-(IC1-PadA1)
- R3 pad 1: Net-(IC1-Pad2) -> Net-(IC1-PadB1)
- R4 pad 2: Net-(IC1-Pad2) -> Net-(IC1-PadB1)
- R5 pad 2: Net-(IC2-Pad1) -> Net-(IC2-PadA1)
- R6 pad 1: Net-(IC2-Pad1) -> Net-(IC2-PadA1)
- R7 pad 2: Net-(IC2-Pad2) -> Net-(IC2-PadB1)
- R8 pad 1: Net-(IC2-Pad2) -> Net-(IC2-PadB1)
Routing:
- net RIJ2: track 72.6 -> 134.7 mm
- net Net-(D8-A): track 0.00 -> 25.4 mm
- net RIJ1: track 91.2 -> 116.4 mm
- net KOLOM3: track 38.9 -> 15.9 mm
- net Net-(D7-A): track 0.00 -> 18.9 mm
- net KOLOM2: track 23.7 -> 7.27 mm
- net Net-(IC2-PadB1): track 0.00 -> 16.1 mm
- net Net-(IC1-PadA1): track 0.00 -> 15.9 mm
- net KOLOM1: track 50.5 -> 35.2 mm
- net ROT2B: track 25.3 -> 10.5 mm
- net KOLOM4: track 0.00 -> 13.4 mm
- net ROT1A: track 25.5 -> 14.6 mm
- net ROT2A: track 20.7 -> 10.5 mm
- net Net-(D3-A): track 2.02 -> 12.1 mm
- net Net-(D1-A): track 2.10 -> 12.1 mm
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